File: hardware/omnibox-v1/sheets/can_fd.kicad_sch (KiCad schematic)
At the start: 40 parts

Commit message: fix(hardware): sync omnibox-v1 with the repaired J2534 V1 KiCad project
Replace the schematic and board with the corrected, single-source-of-truth
version from the upstream J2534 V1 project, and consolidate to one project.

- Schematic + board replaced by the repaired versions (schematic<->PCB relinked
  by symbol UUIDs, 296 (path) links; legal reference designators; library
  prefixes restored on all footprints; USB SuperSpeed pins and MCP2518FD pin 15
  removed to match the fitted footprints; split nets merged: KLINE1/J1962_P7,
  J1850_BUS/J1850_BUSN). Internal project name set to omnibox-v1, company OmniBox.
- Corrected symbols (sym-lib/j2534gen, j2534_local) and footprint libraries.
- Design constraints and net classes aligned to the as-built board (min via
  0.4 mm, min drill 0.2 mm, net-class clearance 0.15 mm).
- Custom DRC rules (.kicad_dru) fixed: '=~' -> '==' (KiCad has no regex; '=='
  does wildcard matching), tightened MCP*CAN / J1850_BUS* patterns, VDDA on the
  host side. Isolation barrier verified with 0 violations, 0 DRC errors.
- Removed the duplicate production/local-finish project; regenerated the
  netlist, consolidated BOM, schematic PDF and Gerbers as omnibox-v1-*.
Parts:
- removed U_CAN4T, U_CAN5T: TJA1463, Package_SO:SOIC-14_3.9x8.7mm_P1.27mm, symbol j2534gen:loc_TJA1463
- added U_CAN4T1, U_CAN5T1: TJA1463, Package_SO:SOIC-14_3.9x8.7mm_P1.27mm, symbol j2534gen:loc_TJA1463
Connections:
- net +3V3_V: now also U_CAN4T1.14 (STB_N), U_CAN4T1.5 (VIO), U_CAN4T1.6 (EN), U_CAN5T1.14 (STB_N), U_CAN5T1.5 (VIO), U_CAN5T1.6 (EN)
- net +5V_V: now also U_CAN4T1.3 (VCC), U_CAN5T1.3 (VCC)
- net CAN4H: now also U_CAN4T1.13 (CANH)
- net CAN4L: now also U_CAN4T1.12 (CANL)
- net CAN5H: now also U_CAN5T1.13 (CANH)
- net CAN5L: now also U_CAN5T1.12 (CANL)
- net GND_V: now also U_CAN4T1.2 (GND), U_CAN5T1.2 (GND); no longer U_CAN4.15 (VSS), U_CAN5.15 (VSS)
- net MCP1_RXCAN: now also U_CAN4T1.4 (RXD)
- net MCP1_TXCAN: now also U_CAN4T1.1 (TXD)
- net MCP2_RXCAN: now also U_CAN5T1.4 (RXD)
- net MCP2_TXCAN: now also U_CAN5T1.1 (TXD)
- net N$27: now also U_CAN4T1.8 (ERR_N)
- net N$28: now also U_CAN4T1.9 (WAKE)
- net N$30: now also U_CAN5T1.8 (ERR_N)
- net N$31: now also U_CAN5T1.9 (WAKE)
- net VBAT_PROT: now also U_CAN4T1.10 (VBAT), U_CAN5T1.10 (VBAT)
Other:
- company: Interface USB-OBD J2534 -> OmniBox
