File: hardware/omnibox-v1/sheets/connector_db25.kicad_sch (KiCad schematic)
At the start: 19 parts, among them J1 DB25_Receptacle_MountingHoles

Commit message: fix(hardware): sync omnibox-v1 with the repaired J2534 V1 KiCad project
Replace the schematic and board with the corrected, single-source-of-truth
version from the upstream J2534 V1 project, and consolidate to one project.

- Schematic + board replaced by the repaired versions (schematic<->PCB relinked
  by symbol UUIDs, 296 (path) links; legal reference designators; library
  prefixes restored on all footprints; USB SuperSpeed pins and MCP2518FD pin 15
  removed to match the fitted footprints; split nets merged: KLINE1/J1962_P7,
  J1850_BUS/J1850_BUSN). Internal project name set to omnibox-v1, company OmniBox.
- Corrected symbols (sym-lib/j2534gen, j2534_local) and footprint libraries.
- Design constraints and net classes aligned to the as-built board (min via
  0.4 mm, min drill 0.2 mm, net-class clearance 0.15 mm).
- Custom DRC rules (.kicad_dru) fixed: '=~' -> '==' (KiCad has no regex; '=='
  does wildcard matching), tightened MCP*CAN / J1850_BUS* patterns, VDDA on the
  host side. Isolation barrier verified with 0 violations, 0 DRC errors.
- Removed the duplicate production/local-finish project; regenerated the
  netlist, consolidated BOM, schematic PDF and Gerbers as omnibox-v1-*.
Parts:
- removed J_PWR: 12V DC 2.5mm, Connector_BarrelJack:BarrelJack_CUI_PJ-102AH_Horizontal, symbol j2534gen:Connector_Barrel_Jack_Switch
- added J_PWR1: 12V DC 2.5mm, Connector_BarrelJack:BarrelJack_CUI_PJ-102AH_Horizontal, symbol j2534gen:Connector_Barrel_Jack_Switch
- J1: footprint Connector_Dsub:DSUB-25_Female_Horizontal_P2.77x2.84mm_EdgePinOffset7.70mm_Housed_MountingHolesOffset9.12mm -> Connector_Dsub:DSUB-25_Socket_Horizontal_P2.77x2.84mm_EdgePinOffset7.70mm_Housed_MountingHolesOffset9.12mm
Connections:
- net GND_V: now also J_PWR1.2
- net VBAT: now also J_PWR1.1
- net J1962_P10 renamed J1850_BUSN
- net J1962_P2 renamed J1850_BUS
- net J1962_P7 renamed KLINE1
Other:
- company: Interface USB-OBD J2534 -> OmniBox
