File: hardware/omnibox-v1/sheets/isolation_barrier.kicad_sch (KiCad schematic)
At the start: 46 parts, among them T1 XFMR_PushPull

Commit message: fix(hardware): sync omnibox-v1 with the repaired J2534 V1 KiCad project
Replace the schematic and board with the corrected, single-source-of-truth
version from the upstream J2534 V1 project, and consolidate to one project.

- Schematic + board replaced by the repaired versions (schematic<->PCB relinked
  by symbol UUIDs, 296 (path) links; legal reference designators; library
  prefixes restored on all footprints; USB SuperSpeed pins and MCP2518FD pin 15
  removed to match the fitted footprints; split nets merged: KLINE1/J1962_P7,
  J1850_BUS/J1850_BUSN). Internal project name set to omnibox-v1, company OmniBox.
- Corrected symbols (sym-lib/j2534gen, j2534_local) and footprint libraries.
- Design constraints and net classes aligned to the as-built board (min via
  0.4 mm, min drill 0.2 mm, net-class clearance 0.15 mm).
- Custom DRC rules (.kicad_dru) fixed: '=~' -> '==' (KiCad has no regex; '=='
  does wildcard matching), tightened MCP*CAN / J1850_BUS* patterns, VDDA on the
  host side. Isolation barrier verified with 0 violations, 0 DRC errors.
- Removed the duplicate production/local-finish project; regenerated the
  netlist, consolidated BOM, schematic PDF and Gerbers as omnibox-v1-*.
Parts:
- removed JP_ISO: SolderJumper_2_Open, Jumper:SolderJumper-2_P1.3mm_Open_Pad1.0x1.5mm, symbol j2534gen:Jumper_SolderJumper_2_Open
- removed LED_V: vert, LED_SMD:LED_0603_1608Metric, symbol j2534gen:Device_LED
- added JP_ISO1: SolderJumper_2_Open, Jumper:SolderJumper-2_P1.3mm_Open_Pad1.0x1.5mm, symbol j2534gen:Jumper_SolderJumper_2_Open
- added LED_V1: vert, LED_SMD:LED_0603_1608Metric, symbol j2534gen:Device_LED
Connections:
- net GND_V: now also LED_V1.1 (K)
- net ISO_PWR_EN: now also JP_ISO1.1 (A)
- net N$14: now also LED_V1.2 (A)
- net VBUS: now also JP_ISO1.2 (B)
Other:
- company: Interface USB-OBD J2534 -> OmniBox
