File: hardware/omnibox-v1/sheets/kline.kicad_sch (KiCad schematic)
At the start: 30 parts

Commit message: fix(hardware): sync omnibox-v1 with the repaired J2534 V1 KiCad project
Replace the schematic and board with the corrected, single-source-of-truth
version from the upstream J2534 V1 project, and consolidate to one project.

- Schematic + board replaced by the repaired versions (schematic<->PCB relinked
  by symbol UUIDs, 296 (path) links; legal reference designators; library
  prefixes restored on all footprints; USB SuperSpeed pins and MCP2518FD pin 15
  removed to match the fitted footprints; split nets merged: KLINE1/J1962_P7,
  J1850_BUS/J1850_BUSN). Internal project name set to omnibox-v1, company OmniBox.
- Corrected symbols (sym-lib/j2534gen, j2534_local) and footprint libraries.
- Design constraints and net classes aligned to the as-built board (min via
  0.4 mm, min drill 0.2 mm, net-class clearance 0.15 mm).
- Custom DRC rules (.kicad_dru) fixed: '=~' -> '==' (KiCad has no regex; '=='
  does wildcard matching), tightened MCP*CAN / J1850_BUS* patterns, VDDA on the
  host side. Isolation barrier verified with 0 violations, 0 DRC errors.
- Removed the duplicate production/local-finish project; regenerated the
  netlist, consolidated BOM, schematic PDF and Gerbers as omnibox-v1-*.
Parts:
- removed C_KL1a, C_KL1b, C_KL2a, C_KL2b, C_KL3a, C_KL3b: 100nF, Capacitor_SMD:C_0603_1608Metric, symbol j2534gen:Device_C
- removed R_KL1a, R_KL2a, R_KL3a: 510, Resistor_SMD:R_0603_1608Metric, symbol j2534gen:Device_R
- removed R_KL1b, R_KL2b, R_KL3b: 47k, Resistor_SMD:R_0603_1608Metric, symbol j2534gen:Device_R
- removed R_KL1c, R_KL1d, R_KL1e, R_KL2c, R_KL2d, R_KL2e, R_KL3c, R_KL3d, R_KL3e: 10k, Resistor_SMD:R_0603_1608Metric, symbol j2534gen:Device_R
- removed R_KL1f, R_KL2f, R_KL3f: 18k, Resistor_SMD:R_0603_1608Metric, symbol j2534gen:Device_R
- added C_KL1a1, C_KL1b1, C_KL2a1, C_KL2b1, C_KL3a1, C_KL3b1: 100nF, Capacitor_SMD:C_0603_1608Metric, symbol j2534gen:Device_C
- added R_KL1a1, R_KL2a1, R_KL3a1: 510, Resistor_SMD:R_0603_1608Metric, symbol j2534gen:Device_R
- added R_KL1b1, R_KL2b1, R_KL3b1: 47k, Resistor_SMD:R_0603_1608Metric, symbol j2534gen:Device_R
- added R_KL1c1, R_KL1d1, R_KL1e1, R_KL2c1, R_KL2d1, R_KL2e1, R_KL3c1, R_KL3d1, R_KL3e1: 10k, Resistor_SMD:R_0603_1608Metric, symbol j2534gen:Device_R
- added R_KL1f1, R_KL2f1, R_KL3f1: 18k, Resistor_SMD:R_0603_1608Metric, symbol j2534gen:Device_R
Connections:
- net +5V_V: now also C_KL1a1.1, C_KL2a1.1, C_KL3a1.1, R_KL1c1.2, R_KL1d1.2, R_KL2c1.2, R_KL2d1.2, R_KL3c1.2, R_KL3d1.2
- net GND_V: now also C_KL1a1.2, C_KL1b1.2, C_KL2a1.2, C_KL2b1.2, C_KL3a1.2, C_KL3b1.2, R_KL1b1.2, R_KL1f1.2, R_KL2b1.2, R_KL2f1.2, R_KL3b1.2, R_KL3f1.2
- net KLINE1: now also R_KL1a1.1
- net KLINE2: now also R_KL2a1.1
- net KLINE3: now also R_KL3a1.1
- net K_RX1_V: now also R_KL1e1.2, R_KL1f1.1
- net K_RX2_V: now also R_KL2e1.2, R_KL2f1.1
- net K_RX3_V: now also R_KL3e1.2, R_KL3f1.1
- net N$32: now also R_KL1d1.1
- net N$33: now also R_KL1e1.1
- net N$34: now also R_KL1b1.1
- net N$35: now also R_KL1c1.1
- net N$36: now also R_KL2d1.1
- net N$37: now also R_KL2e1.1
- net N$38: now also R_KL2b1.1
- net N$39: now also R_KL2c1.1
- net N$40: now also R_KL3d1.1
- net N$41: now also R_KL3e1.1
- net N$42: now also R_KL3b1.1
- net N$43: now also R_KL3c1.1
- net VBAT_PROT: now also C_KL1b1.1, C_KL2b1.1, C_KL3b1.1, R_KL1a1.2, R_KL2a1.2, R_KL3a1.2
Other:
- company: Interface USB-OBD J2534 -> OmniBox
