File: hardware/omnibox-v1/sheets/mcu.kicad_sch (KiCad schematic)
At the start: 33 parts, among them U1 STM32H723ZGTx, Y1 25MHz

Commit message: fix(hardware): sync omnibox-v1 with the repaired J2534 V1 KiCad project
Replace the schematic and board with the corrected, single-source-of-truth
version from the upstream J2534 V1 project, and consolidate to one project.

- Schematic + board replaced by the repaired versions (schematic<->PCB relinked
  by symbol UUIDs, 296 (path) links; legal reference designators; library
  prefixes restored on all footprints; USB SuperSpeed pins and MCP2518FD pin 15
  removed to match the fitted footprints; split nets merged: KLINE1/J1962_P7,
  J1850_BUS/J1850_BUSN). Internal project name set to omnibox-v1, company OmniBox.
- Corrected symbols (sym-lib/j2534gen, j2534_local) and footprint libraries.
- Design constraints and net classes aligned to the as-built board (min via
  0.4 mm, min drill 0.2 mm, net-class clearance 0.15 mm).
- Custom DRC rules (.kicad_dru) fixed: '=~' -> '==' (KiCad has no regex; '=='
  does wildcard matching), tightened MCP*CAN / J1850_BUS* patterns, VDDA on the
  host side. Isolation barrier verified with 0 violations, 0 DRC errors.
- Removed the duplicate production/local-finish project; regenerated the
  netlist, consolidated BOM, schematic PDF and Gerbers as omnibox-v1-*.
Parts:
- removed C_RST, C_VBAT: 100nF, Capacitor_SMD:C_0603_1608Metric, symbol j2534gen:Device_C
- removed JP_BOOT: SolderJumper_2_Open, Jumper:SolderJumper-2_P1.3mm_Open_Pad1.0x1.5mm, symbol j2534gen:Jumper_SolderJumper_2_Open
- removed J_SWD: Conn_02x05_Odd_Even, Connector_PinHeader_1.27mm:PinHeader_2x05_P1.27mm_Vertical, symbol j2534gen:Connector_Generic_Conn_02x05_Odd_Even
- removed LED_H: statut, LED_SMD:LED_0603_1608Metric, symbol j2534gen:Device_LED
- removed LED_PWR: power, LED_SMD:LED_0603_1608Metric, symbol j2534gen:Device_LED
- removed R_BOOT, R_RST: 10k, Resistor_SMD:R_0603_1608Metric, symbol j2534gen:Device_R
- added C_RST1, C_VBAT1: 100nF, Capacitor_SMD:C_0603_1608Metric, symbol j2534gen:Device_C
- added JP_BOOT1: SolderJumper_2_Open, Jumper:SolderJumper-2_P1.3mm_Open_Pad1.0x1.5mm, symbol j2534gen:Jumper_SolderJumper_2_Open
- added J_SWD1: Conn_02x05_Odd_Even, Connector_PinHeader_1.27mm:PinHeader_2x05_P1.27mm_Vertical, symbol j2534gen:Connector_Generic_Conn_02x05_Odd_Even
- added LED_H1: statut, LED_SMD:LED_0603_1608Metric, symbol j2534gen:Device_LED
- added LED_PWR1: alim, LED_SMD:LED_0603_1608Metric, symbol j2534gen:Device_LED
- added R_BOOT1, R_RST1: 10k, Resistor_SMD:R_0603_1608Metric, symbol j2534gen:Device_R
Connections:
- net +3V3_H: now also C_VBAT1.1, JP_BOOT1.2 (B), J_SWD1.1 (Pin_1), R_RST1.2
- net BOOT0: now also JP_BOOT1.1 (A), R_BOOT1.1
- net GND_H: now also C_RST1.2, C_VBAT1.2, J_SWD1.3 (Pin_3), J_SWD1.5 (Pin_5), J_SWD1.9 (Pin_9), LED_H1.1 (K), LED_PWR1.1 (K), R_BOOT1.2
- net N$18: now also LED_H1.2 (A)
- net N$19: now also LED_PWR1.2 (A)
- net NRST: now also C_RST1.1, J_SWD1.10 (Pin_10), R_RST1.1
- net SWCLK: now also J_SWD1.4 (Pin_4)
- net SWDIO: now also J_SWD1.2 (Pin_2)
- net SWD_KEY: now also J_SWD1.7 (Pin_7)
- net SWD_NC: now also J_SWD1.8 (Pin_8)
- net SWO: now also J_SWD1.6 (Pin_6)
Other:
- company: Interface USB-OBD J2534 -> OmniBox
Changed lines of the file:
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@@
 (kicad_sch
-	(version 20231120)(generator "j2534_gen")(generator_version "8.0")
+	(version 20260306)
+	(generator "eeschema")
+	(generator_version "10.0")
 	(paper "A2")
 	(title_block
-		(title "J2534 — mcu")(rev "v1")
-		(company "Interface USB-OBD J2534")
+		(title "J2534 — mcu")
+		(rev "v1")
+		(company "OmniBox")
 	)
