File: hardware/omnibox-v1/sheets/swcan_j1850.kicad_sch (KiCad schematic)
At the start: 40 parts

Commit message: fix(hardware): sync omnibox-v1 with the repaired J2534 V1 KiCad project
Replace the schematic and board with the corrected, single-source-of-truth
version from the upstream J2534 V1 project, and consolidate to one project.

- Schematic + board replaced by the repaired versions (schematic<->PCB relinked
  by symbol UUIDs, 296 (path) links; legal reference designators; library
  prefixes restored on all footprints; USB SuperSpeed pins and MCP2518FD pin 15
  removed to match the fitted footprints; split nets merged: KLINE1/J1962_P7,
  J1850_BUS/J1850_BUSN). Internal project name set to omnibox-v1, company OmniBox.
- Corrected symbols (sym-lib/j2534gen, j2534_local) and footprint libraries.
- Design constraints and net classes aligned to the as-built board (min via
  0.4 mm, min drill 0.2 mm, net-class clearance 0.15 mm).
- Custom DRC rules (.kicad_dru) fixed: '=~' -> '==' (KiCad has no regex; '=='
  does wildcard matching), tightened MCP*CAN / J1850_BUS* patterns, VDDA on the
  host side. Isolation barrier verified with 0 violations, 0 DRC errors.
- Removed the duplicate production/local-finish project; regenerated the
  netlist, consolidated BOM, schematic PDF and Gerbers as omnibox-v1-*.
Parts:
- removed C_J18a, C_J18d: 220pF, Capacitor_SMD:C_0603_1608Metric, symbol j2534gen:Device_C
- removed C_J18c: 1nF, Capacitor_SMD:C_0603_1608Metric, symbol j2534gen:Device_C
- removed D_J18a, D_J18b: B5819W, Diode_SMD:D_SOD-123, symbol j2534gen:loc_D_Schottky
- removed R_J18a: 14k, Resistor_SMD:R_0603_1608Metric, symbol j2534gen:Device_R
- removed R_J18b, R_J18e, R_J18j, R_J18o, R_J18q, R_J18r: 10k, Resistor_SMD:R_0603_1608Metric, symbol j2534gen:Device_R
- removed R_J18c, R_J18k, R_J18m: 33, Resistor_SMD:R_0603_1608Metric, symbol j2534gen:Device_R
- removed R_J18d, R_J18f: 20k, Resistor_SMD:R_0603_1608Metric, symbol j2534gen:Device_R
- removed R_J18g: 6.2k, Resistor_SMD:R_0603_1608Metric, symbol j2534gen:Device_R
- removed R_J18h, R_J18n, R_J18t: 4.7k, Resistor_SMD:R_0603_1608Metric, symbol j2534gen:Device_R
- removed R_J18i: 5.1k, Resistor_SMD:R_0603_1608Metric, symbol j2534gen:Device_R
- removed R_J18l: 15k, Resistor_SMD:R_0603_1608Metric, symbol j2534gen:Device_R
- removed R_J18p, R_J18s: 470k, Resistor_SMD:R_0603_1608Metric, symbol j2534gen:Device_R
- removed R_J18u: 1k, Resistor_SMD:R_0603_1608Metric, symbol j2534gen:Device_R
- removed U_J18A, U_J18B: OPA192, Package_SO:SOIC-8_3.9x4.9mm_P1.27mm, symbol j2534gen:loc_OPA192
- removed U_J18C: LM339, Package_SO:SOIC-14_3.9x8.7mm_P1.27mm, symbol j2534gen:Comparator_LM339
- removed U_SW_CTRL: MCP2518FD-xQBB, Package_SO:SOIC-14_3.9x8.7mm_P1.27mm, symbol j2534gen:Interface_CAN_LIN_MCP2518FD-xQBB
- removed X_SW: 40MHz, Oscillator:Oscillator_SMD_Abracon_ASE-4Pin_3.2x2.5mm, symbol j2534gen:loc_XO
- added C_J18a1, C_J18d1: 220pF, Capacitor_SMD:C_0603_1608Metric, symbol j2534gen:Device_C
- added C_J18c1: 1nF, Capacitor_SMD:C_0603_1608Metric, symbol j2534gen:Device_C
- added D_J18a1, D_J18b1: B5819W, Diode_SMD:D_SOD-123, symbol j2534gen:loc_D_Schottky
- added R_J18a1: 14k, Resistor_SMD:R_0603_1608Metric, symbol j2534gen:Device_R
- added R_J18b1, R_J18e1, R_J18j1, R_J18o1, R_J18q1, R_J18r1: 10k, Resistor_SMD:R_0603_1608Metric, symbol j2534gen:Device_R
- added R_J18c1, R_J18k1, R_J18m1: 33, Resistor_SMD:R_0603_1608Metric, symbol j2534gen:Device_R
- added R_J18d1, R_J18f1: 20k, Resistor_SMD:R_0603_1608Metric, symbol j2534gen:Device_R
- added R_J18g1: 6.2k, Resistor_SMD:R_0603_1608Metric, symbol j2534gen:Device_R
- added R_J18h1, R_J18n1, R_J18t1: 4.7k, Resistor_SMD:R_0603_1608Metric, symbol j2534gen:Device_R
- added R_J18i1: 5.1k, Resistor_SMD:R_0603_1608Metric, symbol j2534gen:Device_R
- added R_J18l1: 15k, Resistor_SMD:R_0603_1608Metric, symbol j2534gen:Device_R
- added R_J18p1, R_J18s1: 470k, Resistor_SMD:R_0603_1608Metric, symbol j2534gen:Device_R
- added R_J18u1: 1k, Resistor_SMD:R_0603_1608Metric, symbol j2534gen:Device_R
- added U_J18A1, U_J18B1: OPA192, Package_SO:SOIC-8_3.9x4.9mm_P1.27mm, symbol j2534gen:loc_OPA192
- added U_J18C1: LM339, Package_SO:SOIC-14_3.9x8.7mm_P1.27mm, symbol j2534gen:Comparator_LM339
- added U_SW_CTRL1: MCP2518FD-xQBB, Package_SO:SOIC-14_3.9x8.7mm_P1.27mm, symbol j2534gen:Interface_CAN_LIN_MCP2518FD-xQBB
- added X_SW1: 40MHz, Oscillator:Oscillator_SMD_Abracon_ASE-4Pin_3.2x2.5mm, symbol j2534gen:loc_XO
Connections:
- net +3V3_V: now also R_J18h1.2, R_J18n1.2, U_SW_CTRL1.14 (VDD), X_SW1.1 (EN), X_SW1.4 (VCC)
- net +5V_V: now also R_J18f1.1, R_J18l1.2, U_J18B1.7 (V+), U_J18C1.10 (-), U_J18C1.3 (V+), U_J18C1.8 (-)
- net CS_MCP3_V: now also U_SW_CTRL1.13 (~{CS})
- net GND_V: now also C_J18a1.2, C_J18c1.2, C_J18d1.2, R_J18b1.2, R_J18e1.2, R_J18g1.2, R_J18j1.2, R_J18o1.2, U_J18A1.4 (V-), U_J18B1.4 (V-), U_J18C1.11 (+), U_J18C1.12 (V-), U_J18C1.9 (+), U_SW_CTRL1.7 (VSS), X_SW1.2 (GND)
- net J1850_BUS: now also C_J18a1.1, R_J18d1.1, R_J18o1.1, R_J18q1.1
- net J1850_BUSN: now also R_J18r1.1
- net J1850_PWMN_DRV: now also R_J18l1.1, R_J18m1.2
- net J1850_PWMP_DRV: now also D_J18b1.1 (K)
- net J1850_PWM_RX_V: now also R_J18n1.1, R_J18s1.1, U_J18C1.1
- net J1850_RX_V: now also R_J18h1.1, R_J18p1.1, U_J18C1.2
- net J1850_TX_V: now also R_J18t1.1, R_J18u1.1
- net J1850_VPW_DRV: now also D_J18a1.1 (K)
- net MCP3_INT_V: now also U_SW_CTRL1.4 (~{INT})
- net N$44: now also U_SW_CTRL1.6 (OSC1), X_SW1.3 (OUT)
- net N$46: now also C_J18c1.1, R_J18t1.2, U_J18A1.3 (IN+)
- net N$47: now also R_J18a1.1, R_J18c1.1, U_J18A1.6 (OUT)
- net N$48: now also R_J18a1.2, R_J18b1.1, U_J18A1.2 (IN-)
- net N$49: now also D_J18a1.2 (A), R_J18c1.2
- net N$50: now also C_J18d1.1, R_J18u1.2, U_J18B1.3 (IN+)
- net N$51: now also R_J18i1.1, R_J18k1.1, U_J18B1.6 (OUT)
- net N$52: now also R_J18i1.2, R_J18j1.1, U_J18B1.2 (IN-)
- net N$53: now also D_J18b1.2 (A), R_J18k1.2
- net N$54: now also R_J18m1.1
- net N$55: now also R_J18f1.2, R_J18g1.1, U_J18C1.4 (-)
- net N$56: now also R_J18r1.2, U_J18C1.6 (-)
- net PWM_CMP_IN: now also R_J18q1.2, R_J18s1.2, U_J18C1.7 (+)
- net SPI_MISO_V: now also U_SW_CTRL1.12 (SDO)
- net SPI_MOSI_V: now also U_SW_CTRL1.11 (SDI)
- net SPI_SCK_V: now also U_SW_CTRL1.10 (SCK)
- net SWCAN_RXCAN: now also U_SW_CTRL1.2 (RXCAN)
- net SWCAN_TXCAN: now also U_SW_CTRL1.1 (TXCAN)
- net VBAT_PROT: now also U_J18A1.7 (V+)
- net VPW_CMP_IN: now also R_J18d1.2, R_J18e1.1, R_J18p1.2, U_J18C1.5 (+)
Other:
- company: Interface USB-OBD J2534 -> OmniBox
