File: hardware/omnibox-v1/sheets/usb_isolated.kicad_sch (KiCad schematic)
At the start: 7 parts

Commit message: fix(hardware): sync omnibox-v1 with the repaired J2534 V1 KiCad project
Replace the schematic and board with the corrected, single-source-of-truth
version from the upstream J2534 V1 project, and consolidate to one project.

- Schematic + board replaced by the repaired versions (schematic<->PCB relinked
  by symbol UUIDs, 296 (path) links; legal reference designators; library
  prefixes restored on all footprints; USB SuperSpeed pins and MCP2518FD pin 15
  removed to match the fitted footprints; split nets merged: KLINE1/J1962_P7,
  J1850_BUS/J1850_BUSN). Internal project name set to omnibox-v1, company OmniBox.
- Corrected symbols (sym-lib/j2534gen, j2534_local) and footprint libraries.
- Design constraints and net classes aligned to the as-built board (min via
  0.4 mm, min drill 0.2 mm, net-class clearance 0.15 mm).
- Custom DRC rules (.kicad_dru) fixed: '=~' -> '==' (KiCad has no regex; '=='
  does wildcard matching), tightened MCP*CAN / J1850_BUS* patterns, VDDA on the
  host side. Isolation barrier verified with 0 violations, 0 DRC errors.
- Removed the duplicate production/local-finish project; regenerated the
  netlist, consolidated BOM, schematic PDF and Gerbers as omnibox-v1-*.
Parts:
- removed J_USB: USB_C_Receptacle, Connector_USB:USB_C_Receptacle_GCT_USB4085, symbol j2534gen:Connector_USB_C_Receptacle
- added J_USB1: USB_C_Receptacle, Connector_USB:USB_C_Receptacle_GCT_USB4085, symbol j2534gen:Connector_USB_C_Receptacle
Connections:
- net GND_H: now also J_USB1.A1 (GND), J_USB1.A12 (GND), J_USB1.B1 (GND), J_USB1.B12 (GND)
- net N$93: now also J_USB1.A5 (CC1)
- net N$94: now also J_USB1.B5 (CC2)
- net USB_DM: now also J_USB1.A7 (D-), J_USB1.B7 (D-)
- net USB_DP: now also J_USB1.A6 (D+), J_USB1.B6 (D+)
- net VBUS: now also J_USB1.A4 (VBUS), J_USB1.A9 (VBUS), J_USB1.B4 (VBUS), J_USB1.B9 (VBUS)
- no-connect marks 11 -> 3
Other:
- company: Interface USB-OBD J2534 -> OmniBox
